File: uC101/Hardware/Panel/output.uc101panel.kicad_pcb (KiCad board)
At the start: 2 copper layers, 100.1 x 99.5 mm, 114 parts, among them J1 Serial / UART, J10 Conn_01x04, J11 Conn_01x04, J2 SPI Header, J3 I2C Header, J4 SAO_Conn, J5 Conn_01x10, J6 Conn_01x10, J7 Conn_01x10, J8 Conn_01x10, J9 Conn_01x04, SW1(D2) SW_Push, SW2(D4) SW_Push, SW3 Rotary_Encoder_Switch

Commit message: some firmware + initial slides
Parts:
- removed the ? at (138.5, 97.7)
- removed the ? at (143.0, 101.5)
- removed the ? at (171.8, 97.7)
- removed the ? at (176.2, 101.5)
- added ?: , holes, F.Cu at (138.4, 97.8)
- added ?: , holes, F.Cu at (143.1, 101.3)
- added ?: , holes, F.Cu at (171.7, 97.8)
- added ?: , holes, F.Cu at (176.3, 101.3)
Changed lines of the file:
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@@
   (module holes
     (layer F.Cu)
-    (at 138.50985 97.65)
+    (at 138.400042 97.8)
     (attr virtual)
     (pad h0 np_thru_hole circle
       (at 0 0)
-      (size 0.6 0.6)
-      (drill 0.6)
+      (size 0.3 0.3)
+      (drill 0.3)
       (layers *.Cu *.Mask))
     (pad h1 np_thru_hole circle
-      (at 1.493452 0)
-      (size 0.6 0.6)
-      (drill 0.6)
+      (at 1.17499 0)
+      (size 0.3 0.3)
+      (drill 0.3)
       (layers *.Cu *.Mask))
     (pad h2 np_thru_hole circle
-      (at 2.986904 0)
-      (size 0.6 0.6)
-      (drill 0.6)
+      (at 2.34998 0)
+      (size 0.3 0.3)
+      (drill 0.3)
       (layers *.Cu *.Mask))
     (pad h3 np_thru_hole circle
-      (at 4.480356 0)
-      (size 0.6 0.6)
-      (drill 0.6)
+      (at 3.52497 0)
+      (size 0.3 0.3)
+      (drill 0.3)
+      (layers *.Cu *.Mask))
+    (pad h4 np_thru_hole circle
+      (at 4.69996 0)
+      (size 0.3 0.3)
+      (drill 0.3)
       (layers *.Cu *.Mask)))
   (gr_line
@@
   (module holes
     (layer F.Cu)
-    (at 142.990254 101.5)
+    (at 143.100063 101.35)
     (attr virtual)
     (pad h0 np_thru_hole circle
       (at 0 0)
-      (size 0.6 0.6)
-      (drill 0.6)
+      (size 0.3 0.3)
+      (drill 0.3)
       (layers *.Cu *.Mask))
     (pad h1 np_thru_hole circle
-      (at -1.493487 0)
-      (size 0.6 0.6)
-      (drill 0.6)
+      (at -1.17502 0)
+      (size 0.3 0.3)
+      (drill 0.3)
       (layers *.Cu *.Mask))
     (pad h2 np_thru_hole circle
-      (at -2.986974 0)
-      (size 0.6 0.6)
-      (drill 0.6)
+      (at -2.35004 0)
+      (size 0.3 0.3)
+      (drill 0.3)
       (layers *.Cu *.Mask))
     (pad h3 np_thru_hole circle
-      (at -4.480461 0)
-      (size 0.6 0.6)
-      (drill 0.6)
+      (at -3.52506 0)
+      (size 0.3 0.3)
+      (drill 0.3)
+      (layers *.Cu *.Mask))
+    (pad h4 np_thru_hole circle
+      (at -4.70008 0)
+      (size 0.3 0.3)
+      (drill 0.3)
       (layers *.Cu *.Mask)))
   (gr_line
@@
   (module holes
     (layer F.Cu)
-    (at 171.759833 97.65)
+    (at 171.650025 97.8)
     (attr virtual)
     (pad h0 np_thru_hole circle
       (at 0 0)
-      (size 0.6 0.6)
-      (drill 0.6)
+      (size 0.3 0.3)
+      (drill 0.3)
       (layers *.Cu *.Mask))
     (pad h1 np_thru_hole circle
-      (at 1.493443 0)
-      (size 0.6 0.6)
-      (drill 0.6)
+      (at 1.174989 0)
+      (size 0.3 0.3)
+      (drill 0.3)
       (layers *.Cu *.Mask))
     (pad h2 np_thru_hole circle
-      (at 2.986886 0)
-      (size 0.6 0.6)
-      (drill 0.6)
+      (at 2.349978 0)
+      (size 0.3 0.3)
+      (drill 0.3)
       (layers *.Cu *.Mask))
     (pad h3 np_thru_hole circle
-      (at 4.480329 0)
-      (size 0.6 0.6)
-      (drill 0.6)
+      (at 3.524967 0)
+      (size 0.3 0.3)
+      (drill 0.3)
+      (layers *.Cu *.Mask))
+    (pad h4 np_thru_hole circle
+      (at 4.699956 0)
+      (size 0.3 0.3)
+      (drill 0.3)
       (layers *.Cu *.Mask)))
   (gr_line
@@
   (module holes
     (layer F.Cu)
-    (at 176.240177 101.5)
+    (at 176.349985 101.35)
     (attr virtual)
     (pad h0 np_thru_hole circle
       (at 0 0)
-      (size 0.6 0.6)
-      (drill 0.6)
+      (size 0.3 0.3)
+      (drill 0.3)
       (layers *.Cu *.Mask))
     (pad h1 np_thru_hole circle
-      (at -1.493443 0)
-      (size 0.6 0.6)
-      (drill 0.6)
+      (at -1.174989 0)
+      (size 0.3 0.3)
+      (drill 0.3)
       (layers *.Cu *.Mask))
     (pad h2 np_thru_hole circle
-      (at -2.986886 0)
-      (size 0.6 0.6)
-      (drill 0.6)
+      (at -2.349978 0)
+      (size 0.3 0.3)
+      (drill 0.3)
       (layers *.Cu *.Mask))
     (pad h3 np_thru_hole circle
-      (at -4.480329 0)
-      (size 0.6 0.6)
-      (drill 0.6)
+      (at -3.524967 0)
+      (size 0.3 0.3)
+      (drill 0.3)
+      (layers *.Cu *.Mask))
+    (pad h4 np_thru_hole circle
+      (at -4.699956 0)
+      (size 0.3 0.3)
+      (drill 0.3)
       (layers *.Cu *.Mask)))
   (gr_line
