File: SAO101/HW/SAO101.sch (KiCad schematic (older format))
At the start: 43 parts, among them J1 USB_B_Micro, J2 SAO_Conn, U1 AMS1117-3.3, U2 MCP23017_SS

Commit message: add csides talk
Parts:
- removed C1: 10u, Capacitor_SMD:C_0805_2012Metric, symbol Device:C
- removed C2: 22u, Capacitor_Tantalum_SMD:CP_EIA-3216-18_Kemet-A, symbol Device:CP1
- removed H1, H2, H3, H4: M3, MountingHole:MountingHole_3.2mm_M3_ISO14580, symbol Mechanical:MountingHole
- removed J1: USB_B_Micro, VNA_Footprints:MicroUSB_Aliexpress, symbol Connector:USB_B_Micro
- removed U1: AMS1117-3.3, Package_TO_SOT_SMD:SOT-223-3_TabPin2, symbol Regulator_Linear:AMS1117-3.3
- renumbered C3 to C1, J2 to J1, U2 to U1
Connections:
- no-connect marks 3 -> 2
Other:
- note added: "SAO Demo Board"
- note removed: "Josh's strange stuff"
- note removed: "SAO 101 Demo Board"
